Commit message: fix 3d

File: public/data/inmoov-local.urdf (robot description, URDF)
Before this commit: robot inmoov, 13 links, 12 joints
Links:
- removed link head_pan_dummy
- removed link head_tilt_dummy
- removed link l_upper_arm_link
- removed link r_upper_arm_link
- added link chestplate_link; visual mesh filename=package://meshes/chest.stl scale=0.001 0.001 0.001
- added link disk_link; visual mesh filename=package://meshes/disk.stl scale=0.001 0.001 0.001
- added link eyesupport_link; visual mesh filename=package://meshes/eyesupport.stl scale=0.001 0.001 0.001
- added link face_link; visual mesh filename=package://meshes/face.stl scale=0.001 0.001 0.001
- added link head_base_link; visual mesh filename=package://meshes/head_base.stl scale=0.001 0.001 0.001
- added link head_tilt_link; visual mesh filename=package://meshes/virtual.stl scale=0.001 0.001 0.001
- added link kinect2_link; visual mesh filename=package://meshes/kinectone.stl scale=0.001 0.001 0.001
- added link l_bicep_link; visual mesh filename=package://meshes/bicep.stl scale=0.001 0.001 0.001
- added link l_bicepcover_link; visual mesh filename=package://meshes/bicepcover.stl scale=0.001 0.001 0.001
- added link l_camera_link; visual mesh filename=package://meshes/camera.stl scale=0.001 0.001 0.001
- added link l_eye_link; visual mesh filename=package://meshes/eye.stl scale=0.001 0.001 0.001
- added link l_eyesupport_link; visual mesh filename=package://meshes/l_eyesupport.stl scale=0.001 0.001 0.001
- added link l_index1_link; visual mesh filename=package://meshes/index3_1.stl scale=0.001 0.001 0.001
- added link l_index2_link; visual mesh filename=package://meshes/index3_2.stl scale=0.001 0.001 0.001
- added link l_index3_link; visual mesh filename=package://meshes/index3_3.stl scale=0.001 0.001 0.001
- added link l_iris_link; visual mesh filename=package://meshes/iris.stl scale=0.001 0.001 0.001
- added link l_middle1_link; visual mesh filename=package://meshes/middle3_1.stl scale=0.001 0.001 0.001
- added link l_middle2_link; visual mesh filename=package://meshes/middle3_2.stl scale=0.001 0.001 0.001
- added link l_middle3_link; visual mesh filename=package://meshes/middle3_3.stl scale=0.001 0.001 0.001
- added link l_pinky1_link; visual mesh filename=package://meshes/l_pinky3_1.stl scale=0.001 0.001 0.001
- added link l_pinky2_link; visual mesh filename=package://meshes/pinky3_2.stl scale=0.001 0.001 0.001
- added link l_pinky3_link; visual mesh filename=package://meshes/pinky3_3.stl scale=0.001 0.001 0.001
- added link l_pinky4_link; visual mesh filename=package://meshes/pinky3_4.stl scale=0.001 0.001 0.001
- added link l_ring1_link; visual mesh filename=package://meshes/l_ring3_1.stl scale=0.001 0.001 0.001
- added link l_ring2_link; visual mesh filename=package://meshes/ring3_2.stl scale=0.001 0.001 0.001
- added link l_ring3_link; visual mesh filename=package://meshes/ring3_3.stl scale=0.001 0.001 0.001
- added link l_ring4_link; visual mesh filename=package://meshes/ring3_4.stl scale=0.001 0.001 0.001
- added link l_shoulder_base_link; visual mesh filename=package://meshes/l_shoulder_base.stl scale=0.001 0.001 0.001
- added link l_thumb1_link; visual mesh filename=package://meshes/l_thumb5_1.stl scale=0.001 0.001 0.001
- added link l_thumb2_link; visual mesh filename=package://meshes/thumb5_2.stl scale=0.001 0.001 0.001
- added link l_thumb3_link; visual mesh filename=package://meshes/thumb5_3.stl scale=0.001 0.001 0.001
- added link left_ear_link; visual mesh filename=package://meshes/earleftv1.stl scale=0.001 0.001 0.001
- added link mid_stomach_link; visual mesh filename=package://meshes/mid_stomach.stl scale=0.001 0.001 0.001
- added link pedestal_link; visual cylinder length=0.94 radius=0.0254
- added link r_bicep_link; visual mesh filename=package://meshes/bicep.stl scale=0.001 0.001 0.001
- added link r_bicepcover_link; visual mesh filename=package://meshes/bicepcover.stl scale=0.001 0.001 0.001
- added link r_camera_link; visual mesh filename=package://meshes/camera.stl scale=0.001 0.001 0.001
- added link r_eye_link; visual mesh filename=package://meshes/eye.stl scale=0.001 0.001 0.001
- added link r_eyesupport_link; visual mesh filename=package://meshes/r_eyesupport.stl scale=0.001 0.001 0.001
- added link r_index1_link; visual mesh filename=package://meshes/index3_1.stl scale=0.001 0.001 0.001
- added link r_index2_link; visual mesh filename=package://meshes/index3_2.stl scale=0.001 0.001 0.001
- added link r_index3_link; visual mesh filename=package://meshes/index3_3.stl scale=0.001 0.001 0.001
- added link r_iris_link; visual mesh filename=package://meshes/iris.stl scale=0.001 0.001 0.001
- added link r_middle1_link; visual mesh filename=package://meshes/middle3_1.stl scale=0.001 0.001 0.001
- added link r_middle2_link; visual mesh filename=package://meshes/middle3_2.stl scale=0.001 0.001 0.001
- added link r_middle3_link; visual mesh filename=package://meshes/middle3_3.stl scale=0.001 0.001 0.001
- added link r_pinky1_link; visual mesh filename=package://meshes/r_pinky3_1.stl scale=0.001 0.001 0.001
- added link r_pinky2_link; visual mesh filename=package://meshes/pinky3_2.stl scale=0.001 0.001 0.001
- added link r_pinky3_link; visual mesh filename=package://meshes/pinky3_3.stl scale=0.001 0.001 0.001
- added link r_pinky4_link; visual mesh filename=package://meshes/pinky3_4.stl scale=0.001 0.001 0.001
- added link r_ring1_link; visual mesh filename=package://meshes/r_ring3_1.stl scale=0.001 0.001 0.001
- added link r_ring2_link; visual mesh filename=package://meshes/ring3_2.stl scale=0.001 0.001 0.001
- added link r_ring3_link; visual mesh filename=package://meshes/ring3_3.stl scale=0.001 0.001 0.001
- added link r_ring4_link; visual mesh filename=package://meshes/ring3_4.stl scale=0.001 0.001 0.001
- added link r_shoulder_base_link; visual mesh filename=package://meshes/r_shoulder_base.stl scale=0.001 0.001 0.001
- added link r_thumb1_link; visual mesh filename=package://meshes/r_thumb5_1.stl scale=0.001 0.001 0.001
- added link r_thumb2_link; visual mesh filename=package://meshes/thumb5_2.stl scale=0.001 0.001 0.001
- added link r_thumb3_link; visual mesh filename=package://meshes/thumb5_3.stl scale=0.001 0.001 0.001
- added link right_ear_link; visual mesh filename=package://meshes/earrightv1.stl scale=0.001 0.001 0.001
- added link skull_link; visual mesh filename=package://meshes/skull.stl scale=0.001 0.001 0.001
- added link top_stomach_link; visual mesh filename=package://meshes/top_stomach.stl scale=0.001 0.001 0.001
- added link torso_link; visual mesh filename=package://meshes/torso.stl scale=0.001 0.001 0.001
- added link world
- link base_link: geometry visual cylinder length=0.11 radius=0.26
Joints:
- added joint base_to_pedestal_link: type fixed, parent base_link, child pedestal_link, origin xyz=0 0 0 rpy=0 0 0
- added joint chestplate_joint: type fixed, parent torso_link, child chestplate_link, origin xyz=0.042 0 0.025 rpy=0 0 0
- added joint disk_joint: type fixed, parent top_stomach_link, child disk_link, origin xyz=0.046 0 0.09 rpy=0 0 0
- added joint eyes_pan_joint: type revolute, parent eyesupport_link, child r_eyesupport_link, origin xyz=0 0.033 -0.0036 rpy=0 0 0, axis 0 0 1, limit lower=-0.5 upper=0.5 effort=1000 velocity=1.0
- added joint eyes_tilt_joint: type revolute, parent face_link, child eyesupport_link, origin xyz=0 0 0 rpy=0 0 0, axis 0 1 0, limit lower=-0.5 upper=0.5 effort=1000 velocity=1.0
- added joint face_joint: type fixed, parent skull_link, child face_link, origin xyz=0.0637 0 0.079 rpy=0 0 0
- added joint fixed: type fixed, parent world, child base_link, origin xyz=0 0 0 rpy=0 0 0
- added joint kinect2_joint: type fixed, parent torso_link, child kinect2_link, origin xyz=0 0 0.066 rpy=-1.57 0 -1.57
- added joint l_bicepcover_joint: type fixed, parent l_bicep_link, child l_bicepcover_link, origin xyz=0 0 0 rpy=0 0 0
- added joint l_camera_joint: type fixed, parent l_eyesupport_link, child l_camera_link, origin xyz=-0.001 0 0 rpy=0 0 0
- added joint l_eye_joint: type fixed, parent l_eyesupport_link, child l_eye_link, origin xyz=0.003 0 0 rpy=0 0 0
- added joint l_eye_pan_joint: type revolute, parent eyesupport_link, child l_eyesupport_link, origin xyz=0 -0.033 -0.0036 rpy=0 0 0, axis 0 0 1, limit lower=-0.5 upper=0.5 effort=1000 velocity=1.0
- added joint l_index1_joint: type revolute, parent l_hand_link, child l_index1_link, origin xyz=-0.0015 -0.0342 -0.119 rpy=-0.1 0 0, axis 0 1 0, limit lower=-1.2 upper=1.2 effort=1000 velocity=1.0
- added joint l_index3_joint: type revolute, parent l_index2_link, child l_index3_link, origin xyz=0 0 -0.024 rpy=0 0 0, axis 0 1 0, limit lower=-1.2 upper=1.2 effort=1000 velocity=1.0
- added joint l_index_joint: type revolute, parent l_index1_link, child l_index2_link, origin xyz=0 0.001 -0.03595 rpy=0 0 0, axis 0 1 0, limit lower=-1.2 upper=1.2 effort=1000 velocity=1.0
- added joint l_iris_joint: type fixed, parent l_eyesupport_link, child l_iris_link, origin xyz=0.0061 0 0 rpy=0 0 0
- added joint l_middle1_joint: type revolute, parent l_hand_link, child l_middle1_link, origin xyz=-0.00175 -0.007 -0.12325 rpy=0 0 0, axis 0 1 0, limit lower=-1.2 upper=1.2 effort=1000 velocity=1.0
- added joint l_middle3_joint: type revolute, parent l_middle2_link, child l_middle3_link, origin xyz=0 0.0005 -0.0259 rpy=0 0 0, axis 0 1 0, limit lower=-1.2 upper=1.2 effort=1000 velocity=1.0
- added joint l_middle_joint: type revolute, parent l_middle1_link, child l_middle2_link, origin xyz=0 0 -0.0389 rpy=0 0 0, axis 0 1 0, limit lower=-1.2 upper=1.2 effort=1000 velocity=1.0
- added joint l_pinky1_joint: type revolute, parent l_hand_link, child l_pinky1_link, origin xyz=0 0.0270 -0.0555 rpy=-0.7 0 0, axis 0 0 1, limit lower=-1.2 upper=1.2 effort=1000 velocity=1.0
- added joint l_pinky3_joint: type revolute, parent l_pinky2_link, child l_pinky3_link, origin xyz=0 0.0005 -0.031 rpy=0 0 0, axis 0 1 0, limit lower=-1.2 upper=1.2 effort=1000 velocity=1.0
- added joint l_pinky4_joint: type revolute, parent l_pinky3_link, child l_pinky4_link, origin xyz=0 0.0004 -0.0208 rpy=0 0 0, axis 0 1 0, limit lower=-1.2 upper=1.2 effort=1000 velocity=1.0
- added joint l_pinky_joint: type revolute, parent l_pinky1_link, child l_pinky2_link, origin xyz=0 0.046 -0.0228 rpy=0.93 0 0, axis 0 1 0, limit lower=-1.2 upper=1.2 effort=1000 velocity=1.0
- added joint l_ring1_joint: type revolute, parent l_hand_link, child l_ring1_link, origin xyz=0 0.00705 -0.0794 rpy=-0.7 0 0, axis 0 0 1, limit lower=-1.2 upper=1.2 effort=1000 velocity=1.0
- added joint l_ring3_joint: type revolute, parent l_ring2_link, child l_ring3_link, origin xyz=0 0.0005 -0.0345 rpy=0 0 0, axis 0 1 0, limit lower=-1.2 upper=1.2 effort=1000 velocity=1.0
- added joint l_ring4_joint: type revolute, parent l_ring3_link, child l_ring4_link, origin xyz=0 0.0004 -0.0229 rpy=0 0 0, axis 0 1 0, limit lower=-1.2 upper=1.2 effort=1000 velocity=1.0
- added joint l_ring_joint: type revolute, parent l_ring1_link, child l_ring2_link, origin xyz=0.00126 0.0351 -0.0166 rpy=0.7775 0 0, axis 0 1 0, limit lower=-1.2 upper=1.2 effort=1000 velocity=1.0
- added joint l_thumb1_joint: type revolute, parent l_hand_link, child l_thumb1_link, origin xyz=0 -0.029 -0.0577 rpy=-0.1 0 0, axis 0 0 1, limit lower=-1.2 upper=1.2 effort=1000 velocity=1.0
- added joint l_thumb3_joint: type revolute, parent l_thumb2_link, child l_thumb3_link, origin xyz=0 0 -0.035 rpy=0 0 0, axis 0 1 0, limit lower=-1.2 upper=1.2 effort=1000 velocity=1.0
- added joint l_thumb_joint: type revolute, parent l_thumb1_link, child l_thumb2_link, origin xyz=-0.00052 -0.02725 -0.013 rpy=-0.825 -0.1 -0.3, axis 0 1 0, limit lower=-1.2 upper=1.2 effort=1000 velocity=1.0
- added joint l_upper_arm_roll_joint: type revolute, parent l_shoulder_link, child l_bicep_link, origin xyz=0 0.066 -0.060 rpy=0 0 0, axis 0 0 1, limit lower=-1.57 upper=1.57 effort=1000 velocity=1.0
- added joint left_ear_joint: type fixed, parent head_link, child left_ear_link, origin xyz=0.035 0.056 0.0437 rpy=0 0 0
- added joint pedestal_to_mid_stomach_joint: type fixed, parent pedestal_link, child mid_stomach_link, origin xyz=0 0 0 rpy=0 0 0
- added joint r_bicepcover_joint: type fixed, parent r_bicep_link, child r_bicepcover_link, origin xyz=0 0 0 rpy=0 0 0
- added joint r_camera_joint: type fixed, parent r_eyesupport_link, child r_camera_link, origin xyz=-0.001 0 0 rpy=0 0 0
- added joint r_eye_joint: type fixed, parent r_eyesupport_link, child r_eye_link, origin xyz=0.003 0 0 rpy=0 0 0
- added joint r_index1_joint: type revolute, parent r_hand_link, child r_index1_link, origin xyz=-0.0015 0.0342 -0.119 rpy=0.1 0 0, axis 0 1 0, limit lower=-1.2 upper=1.2 effort=1000 velocity=1.0
- added joint r_index3_joint: type revolute, parent r_index2_link, child r_index3_link, origin xyz=0 0 -0.024 rpy=0 0 0, axis 0 1 0, limit lower=-1.2 upper=1.2 effort=1000 velocity=1.0
- added joint r_index_joint: type revolute, parent r_index1_link, child r_index2_link, origin xyz=0 0.001 -0.03595 rpy=0 0 0, axis 0 1 0, limit lower=-1.2 upper=1.2 effort=1000 velocity=1.0
- added joint r_iris_joint: type fixed, parent r_eyesupport_link, child r_iris_link, origin xyz=0.0061 0 0 rpy=0 0 0
- added joint r_middle1_joint: type revolute, parent r_hand_link, child r_middle1_link, origin xyz=-0.00175 0.007 -0.12325 rpy=0 0 0, axis 0 1 0, limit lower=-1.2 upper=1.2 effort=1000 velocity=1.0
- added joint r_middle3_joint: type revolute, parent r_middle2_link, child r_middle3_link, origin xyz=0 0.0005 -0.0259 rpy=0 0 0, axis 0 1 0, limit lower=-1.2 upper=1.2 effort=1000 velocity=1.0
- added joint r_middle_joint: type revolute, parent r_middle1_link, child r_middle2_link, origin xyz=0 0 -0.0389 rpy=0 0 0, axis 0 1 0, limit lower=-1.2 upper=1.2 effort=1000 velocity=1.0
- added joint r_pinky1_joint: type revolute, parent r_hand_link, child r_pinky1_link, origin xyz=0 -0.0270 -0.0555 rpy=0.7 0 0, axis 0 0 1, limit lower=-1.2 upper=1.2 effort=1000 velocity=1.0
- added joint r_pinky3_joint: type revolute, parent r_pinky2_link, child r_pinky3_link, origin xyz=0 0.0005 -0.031 rpy=0 0 0, axis 0 1 0, limit lower=-1.2 upper=1.2 effort=1000 velocity=1.0
- added joint r_pinky4_joint: type revolute, parent r_pinky3_link, child r_pinky4_link, origin xyz=0 0.0004 -0.0208 rpy=0 0 0, axis 0 1 0, limit lower=-1.2 upper=1.2 effort=1000 velocity=1.0
- added joint r_pinky_joint: type revolute, parent r_pinky1_link, child r_pinky2_link, origin xyz=0 -0.046 -0.0228 rpy=-0.93 0 0, axis 0 1 0, limit lower=-1.2 upper=1.2 effort=1000 velocity=1.0
- added joint r_ring1_joint: type revolute, parent r_hand_link, child r_ring1_link, origin xyz=0 -0.00705 -0.0794 rpy=0.7 0 0, axis 0 0 1, limit lower=-1.2 upper=1.2 effort=1000 velocity=1.0
- added joint r_ring3_joint: type revolute, parent r_ring2_link, child r_ring3_link, origin xyz=0 0.0005 -0.0345 rpy=0 0 0, axis 0 1 0, limit lower=-1.2 upper=1.2 effort=1000 velocity=1.0
- added joint r_ring4_joint: type revolute, parent r_ring3_link, child r_ring4_link, origin xyz=0 0.0004 -0.0229 rpy=0 0 0, axis 0 1 0, limit lower=-1.2 upper=1.2 effort=1000 velocity=1.0
- added joint r_ring_joint: type revolute, parent r_ring1_link, child r_ring2_link, origin xyz=0.00126 -0.0351 -0.0166 rpy=-0.7775 0 0, axis 0 1 0, limit lower=-1.2 upper=1.2 effort=1000 velocity=1.0
- added joint r_thumb1_joint: type revolute, parent r_hand_link, child r_thumb1_link, origin xyz=0 0.029 -0.0577 rpy=0.1 0 0, axis 0 0 1, limit lower=-1.2 upper=1.2 effort=1000 velocity=1.0
- added joint r_thumb3_joint: type revolute, parent r_thumb2_link, child r_thumb3_link, origin xyz=0 0 -0.035 rpy=0 0 0, axis 0 1 0, limit lower=-1.2 upper=1.2 effort=1000 velocity=1.0
- added joint r_thumb_joint: type revolute, parent r_thumb1_link, child r_thumb2_link, origin xyz=-0.00052 0.02725 -0.013 rpy=0.825 -0.1 0.3, axis 0 1 0, limit lower=-1.2 upper=1.2 effort=1000 velocity=1.0
- added joint r_upper_arm_roll_joint: type revolute, parent r_shoulder_link, child r_bicep_link, origin xyz=0 -0.066 -0.060 rpy=0 0 0, axis 0 0 1, limit lower=-1.57 upper=1.57 effort=1000 velocity=1.0
- added joint right_ear_joint: type fixed, parent head_link, child right_ear_link, origin xyz=0.035 -0.056 0.0437 rpy=0 0 0
- added joint skull_joint: type fixed, parent head_link, child skull_link, origin xyz=0.044 0 -0.0245 rpy=0 0 0
- added joint waist_pan_joint: type revolute, parent mid_stomach_link, child top_stomach_link, origin xyz=0 0 1.152 rpy=0 0 0, axis 0 0 1, limit lower=-0.6 upper=0.6 effort=1000 velocity=1.0
- added joint waist_roll_joint: type revolute, parent top_stomach_link, child torso_link, origin xyz=0 0 0.11 rpy=0 0 0, axis 1 0 0, limit lower=-0.5 upper=0.5 effort=1000 velocity=1.0
- joint head_pan_joint: child head_pan_dummy -> head_link; limit lower=-1.57 upper=1.57 effort=5 velocity=1 -> lower=-1.2 upper=1.2 effort=1000 velocity=1.0; origin xyz=0 0 0 rpy=0 0 0 -> xyz=0 0 0.0245 rpy=0 0 0; parent head_link -> head_base_link
- joint head_roll_joint: child head_link -> head_tilt_link; limit lower=-1.57 upper=1.57 effort=10 velocity=1 -> lower=-0.6 upper=0.6 effort=1000 velocity=1.0; origin xyz=0.0 0.0 0.4 rpy=0 0 0 -> xyz=-0.0315 -0.001 0.4551 rpy=0 0 3.1415; parent base_link -> torso_link
- joint head_tilt_joint: child head_tilt_dummy -> head_base_link; limit lower=-1.57 upper=1.57 effort=5 velocity=1 -> lower=-0.6 upper=0.6 effort=1000 velocity=1.0; origin xyz=0 0 0 rpy=0 0 0 -> xyz=0 0 0 rpy=0 0 3.1415; parent head_link -> head_tilt_link
- joint jaw_joint: axis 1 0 0 -> 0 1 0; limit lower=0 upper=0.6 effort=5 velocity=1 -> lower=0 upper=0.8 effort=1000 velocity=1.0; origin xyz=0.0 0.0 -0.08 rpy=0 0 0 -> xyz=0.0375 0.0005 0.0437 rpy=0 0.09 0
- joint l_elbow_flex_joint: axis 0 0 1 -> 0 1 0; limit lower=0 upper=2.09 effort=10 velocity=1 -> lower=0 upper=2.09 effort=1000 velocity=1.0; origin xyz=0.18 0.0 0.0 rpy=0 0 0 -> xyz=-0.0278 0 -0.2235 rpy=0 0 0; parent l_upper_arm_link -> l_bicep_link
- joint l_shoulder_lift_joint: axis 0 0 1 -> 0 1 0; child l_upper_arm_link -> l_shoulder_link; limit lower=-1.57 upper=1.57 effort=15 velocity=1 -> lower=-1.57 upper=1.57 effort=1000 velocity=1.0; origin xyz=0.1 0.0 0.0 rpy=0 0 0 -> xyz=0 0.012 -0.04 rpy=0 0 0; parent l_shoulder_link -> l_shoulder_base_link
- joint l_shoulder_out_joint: axis 0 1 0 -> 1 0 0; child l_shoulder_link -> l_shoulder_base_link; limit lower=-1.57 upper=1.57 effort=15 velocity=1 -> lower=-1.2 upper=1.2 effort=1000 velocity=1.0; origin xyz=0.2 0.0 0.2 rpy=0 0 0 -> xyz=0 0.143 0.298 rpy=0 0 0; parent base_link -> torso_link
- joint l_wrist_roll_joint: axis 1 0 0 -> 0 0 1; limit lower=-3.14 upper=3.14 effort=10 velocity=1 -> lower=-3.14 upper=3.14 effort=1000 velocity=1.0; origin xyz=0.18 0.0 0.0 rpy=0 0 0 -> xyz=-0.0144 -0.01 -0.2885 rpy=0 0 0
- joint r_elbow_flex_joint: axis 0 0 1 -> 0 1 0; limit lower=0 upper=2.09 effort=10 velocity=1 -> lower=0 upper=2.09 effort=1000 velocity=1.0; origin xyz=-0.18 0.0 0.0 rpy=0 0 0 -> xyz=-0.0278 0 -0.2235 rpy=0 0 0; parent r_upper_arm_link -> r_bicep_link
- joint r_shoulder_lift_joint: axis 0 0 1 -> 0 1 0; child r_upper_arm_link -> r_shoulder_link; limit lower=-1.57 upper=1.57 effort=15 velocity=1 -> lower=-1.57 upper=1.57 effort=1000 velocity=1.0; origin xyz=-0.1 0.0 0.0 rpy=0 0 0 -> xyz=0 -0.012 -0.04 rpy=0 0 0; parent r_shoulder_link -> r_shoulder_base_link
- joint r_shoulder_out_joint: axis 0 1 0 -> 1 0 0; child r_shoulder_link -> r_shoulder_base_link; limit lower=-1.57 upper=1.57 effort=15 velocity=1 -> lower=-1.2 upper=1.2 effort=1000 velocity=1.0; origin xyz=-0.2 0.0 0.2 rpy=0 0 0 -> xyz=0 -0.143 0.298 rpy=0 0 0; parent base_link -> torso_link
- joint r_wrist_roll_joint: axis 1 0 0 -> 0 0 1; limit lower=-3.14 upper=3.14 effort=10 velocity=1 -> lower=-3.14 upper=3.14 effort=1000 velocity=1.0; origin xyz=-0.18 0.0 0.0 rpy=0 0 0 -> xyz=-0.0144 0.01 -0.2885 rpy=0 0 0
