Commit message: before codex

File: public/data/inmoov-local.urdf (robot description, URDF)
Before this commit: robot inmoov_local_fixed, 72 links, 71 joints
Links:
- added link l_cover_handpinky_link; visual mesh filename=package://meshes/l_cover_handpinky.stl scale=0.001 0.001 0.001
- added link l_cover_handring_link; visual mesh filename=package://meshes/l_cover_handring.stl scale=0.001 0.001 0.001
- added link l_cover_index_link; visual mesh filename=package://meshes/l_cover_index.stl scale=0.001 0.001 0.001
- added link l_cover_middle_link; visual mesh filename=package://meshes/l_cover_middle.stl scale=0.001 0.001 0.001
- added link l_cover_pinky_link; visual mesh filename=package://meshes/l_cover_pinky.stl scale=0.001 0.001 0.001
- added link l_cover_ring_link; visual mesh filename=package://meshes/l_cover_ring.stl scale=0.001 0.001 0.001
- added link l_cover_thumb_link; visual mesh filename=package://meshes/l_cover_thumb.stl scale=0.001 0.001 0.001
- added link l_handcover_link; visual mesh filename=package://meshes/l_cover_hand.stl scale=0.001 0.001 0.001
- added link r_cover_handpinky_link; visual mesh filename=package://meshes/r_cover_handpinky.stl scale=0.001 0.001 0.001
- added link r_cover_handring_link; visual mesh filename=package://meshes/r_cover_handring.stl scale=0.001 0.001 0.001
- added link r_cover_index_link; visual mesh filename=package://meshes/r_cover_index.stl scale=0.001 0.001 0.001
- added link r_cover_middle_link; visual mesh filename=package://meshes/r_cover_middle.stl scale=0.001 0.001 0.001
- added link r_cover_pinky_link; visual mesh filename=package://meshes/r_cover_pinky.stl scale=0.001 0.001 0.001
- added link r_cover_ring_link; visual mesh filename=package://meshes/r_cover_ring.stl scale=0.001 0.001 0.001
- added link r_cover_thumb_link; visual mesh filename=package://meshes/r_cover_thumb.stl scale=0.001 0.001 0.001
- added link r_handcover_link; visual mesh filename=package://meshes/r_cover_hand.stl scale=0.001 0.001 0.001
Joints:
- added joint l_cover_handpinky_joint: type fixed, parent l_pinky1_link, child l_cover_handpinky_link, origin xyz=0.01 0.02025 -0.0071 rpy=0.7 0 0
- added joint l_cover_handring_joint: type fixed, parent l_ring1_link, child l_cover_handring_link, origin xyz=0.009 0.015 -0.0008 rpy=0.7 0 0
- added joint l_cover_index_joint: type fixed, parent l_index1_link, child l_cover_index_link, origin xyz=0.0071 0 -0.012 rpy=0 -0.05 0
- added joint l_cover_middle_joint: type fixed, parent l_middle1_link, child l_cover_middle_link, origin xyz=0.0071 0 -0.012 rpy=0 0.05 0
- added joint l_cover_pinky_joint: type fixed, parent l_pinky2_link, child l_cover_pinky_link, origin xyz=0.005 0 -0.0105 rpy=-0.1 0.05 0
- added joint l_cover_ring_joint: type fixed, parent l_ring2_link, child l_cover_ring_link, origin xyz=0.005 0 -0.011 rpy=-0.1 0.05 0
- added joint l_cover_thumb_joint: type fixed, parent l_thumb1_link, child l_cover_thumb_link, origin xyz=0.01 -0.02125 0.0047 rpy=-0.05 0 0
- added joint l_handcover_joint: type fixed, parent l_hand_link, child l_handcover_link, origin xyz=0.009 -0.0192 -0.0977 rpy=0 0 0
- added joint r_cover_handpinky_joint: type fixed, parent r_pinky1_link, child r_cover_handpinky_link, origin xyz=0.01 -0.02025 -0.0071 rpy=-0.7 0 0
- added joint r_cover_handring_joint: type fixed, parent r_ring1_link, child r_cover_handring_link, origin xyz=0.009 -0.015 -0.0008 rpy=-0.7 0 0
- added joint r_cover_index_joint: type fixed, parent r_index1_link, child r_cover_index_link, origin xyz=0.0071 0 -0.012 rpy=0 0.05 0
- added joint r_cover_middle_joint: type fixed, parent r_middle1_link, child r_cover_middle_link, origin xyz=0.0071 0 -0.012 rpy=0 -0.05 0
- added joint r_cover_pinky_joint: type fixed, parent r_pinky2_link, child r_cover_pinky_link, origin xyz=0.005 0 -0.0105 rpy=0.1 -0.05 0
- added joint r_cover_ring_joint: type fixed, parent r_ring2_link, child r_cover_ring_link, origin xyz=0.005 0 -0.011 rpy=0.1 -0.05 0
- added joint r_cover_thumb_joint: type fixed, parent r_thumb1_link, child r_cover_thumb_link, origin xyz=0.01 0.02125 0.0047 rpy=0.05 0 0
- added joint r_handcover_joint: type fixed, parent r_hand_link, child r_handcover_link, origin xyz=0.009 0.0192 -0.0977 rpy=0 0 0
